Commit message: Create urdf folder and move urdf files there. Also, use xacro variables for radian to degrees convertion.

File: urdf/comau.urdf.xacro (robot description, xacro)
@@ -2,9 +2,11 @@
 <robot xmlns:xacro="http://ros.org/wiki/xacro" name="comau">
     <xacro:include filename="materials.xacro"/>
+    <xacro:property name="r2d" value="${pi/180}"/>
+    <xacro:property name="meshes_path" value="package://comau_racer5_080_description/meshes"/>
     <link name="base_link">
         <visual>
             <origin xyz="0 0 0" rpy="0 0 0"/>
             <geometry>
-                <mesh filename="package://comau_racer5_080_description/meshes/Base.stl" scale="0.001 0.001 0.001"/>
+                <mesh filename="${meshes_path}/Base.stl" scale="0.001 0.001 0.001"/>
             </geometry>
             <material name="grey"/>
@@ -15,5 +17,5 @@
             <origin xyz="0 0 0.19" rpy="0 0 0"/>
             <geometry>
-                <mesh filename="package://comau_racer5_080_description/meshes/Q1.stl" scale="0.001 0.001 0.001"/>
+                <mesh filename="${meshes_path}/Q1.stl" scale="0.001 0.001 0.001"/>
             </geometry>
             <material name="grey"/>
@@ -24,5 +26,5 @@
        <parent link="base_link"/>
        <child link="q1_link"/>
-       <limit lower="-2.9671" upper="2.9671" effort="0.0" velocity="6.98131701"/>
+       <limit lower="-${r2d*170}" upper="${r2d*170}" effort="0.0" velocity="${r2d*400}"/>
     </joint>
     <link name="q2_link">
@@ -30,5 +32,5 @@
             <origin xyz="0 0 0" rpy="0 0 0"/>
             <geometry>
-                <mesh filename="package://comau_racer5_080_description/meshes/Q2.stl" scale="0.001 0.001 0.001"/>
+                <mesh filename="${meshes_path}/Q2.stl" scale="0.001 0.001 0.001"/>
             </geometry>
             <material name="grey"/>
@@ -40,5 +42,5 @@
        <parent link="q1_link"/>
        <child link="q2_link"/>
-       <limit lower="-1.48352986" upper="2.35619449" effort="0.0" velocity="6.28318531"/>
+       <limit lower="-${r2d*85}" upper="${r2d*135}" effort="0.0" velocity="${r2d*360}"/>
     </joint>
     <link name="q3_link">
@@ -46,5 +48,5 @@
             <origin xyz="0 0 0" rpy="0 0 0"/>
             <geometry>
-                <mesh filename="package://comau_racer5_080_description/meshes/Q3.stl" scale="0.001 0.001 0.001"/>
+                <mesh filename="${meshes_path}/Q3.stl" scale="0.001 0.001 0.001"/>
             </geometry>
             <material name="grey"/>
@@ -56,5 +58,5 @@
        <parent link="q2_link"/>
        <child link="q3_link"/>
-       <limit lower="-2.70526034" upper="1.57079633" effort="0.0" velocity="6.98131701"/>
+       <limit lower="-${r2d*155}" upper="${r2d*90}" effort="0.0" velocity="${r2d*400}"/>
     </joint>
     <link name="q4_link">
@@ -62,5 +64,5 @@
             <origin xyz="0 0 0" rpy="0 0 0"/>
             <geometry>
-                <mesh filename="package://comau_racer5_080_description/meshes/Q4.stl" scale="0.001 0.001 0.001"/>
+                <mesh filename="${meshes_path}/Q4.stl" scale="0.001 0.001 0.001"/>
             </geometry>
             <material name="grey"/>
@@ -72,5 +74,5 @@
        <parent link="q3_link"/>
        <child link="q4_link"/>
-       <limit lower="-3.4906585" upper="3.4906585" effort="0.0" velocity="8.72664626"/>
+       <limit lower="-${r2d*200}" upper="${r2d*200}" effort="0.0" velocity="${r2d*500}"/>
     </joint>
     <link name="q5_link">
@@ -78,5 +80,5 @@
             <origin xyz="0 0 0" rpy="0 0 0"/>
             <geometry>
-                <mesh filename="package://comau_racer5_080_description/meshes/Q5.stl" scale="0.001 0.001 0.001"/>
+                <mesh filename="${meshes_path}/Q5.stl" scale="0.001 0.001 0.001"/>
             </geometry>
             <material name="grey"/>
@@ -88,5 +90,5 @@
        <parent link="q4_link"/>
        <child link="q5_link"/>
-       <limit lower="-2.18166156" upper="2.18166156" effort="0.0" velocity="8.72664626"/>
+       <limit lower="-${r2d*125}" upper="${r2d*125}" effort="0.0" velocity="${r2d*500}"/>
     </joint>
     <link name="q6_link">
@@ -94,5 +96,5 @@
             <origin xyz="0 0 0" rpy="0 0 0"/>
             <geometry>
-                <mesh filename="package://comau_racer5_080_description/meshes/Q6.stl" scale="0.001 0.001 0.001"/>
+                <mesh filename="${meshes_path}/Q6.stl" scale="0.001 0.001 0.001"/>
             </geometry>
             <material name="grey"/>
@@ -104,5 +106,5 @@
        <parent link="q5_link"/>
        <child link="q6_link"/>
-       <limit lower="-47.1238898" upper="47.1238898" effort="0.0" velocity="13.962634"/>
+       <limit lower="-${r2d*2700}" upper="${r2d*2700}" effort="0.0" velocity="${r2d*800}"/>
     </joint>
 </robot>

Commit message: Set up gazebo simulation (not working yet)

File: urdf/comau.urdf.xacro (robot description, xacro)
@@ -1,5 +1,14 @@
 <?xml version="1.0"?>
-<robot xmlns:xacro="http://ros.org/wiki/xacro" name="comau">
-    <xacro:include filename="materials.xacro"/>
+<robot xmlns:xacro="http://www.ros.org/wiki/xacro" name="comau">
+    <xacro:include filename="$(find comau_racer5_080_description)/urdf/materials.xacro"/>
+    <!-- <xacro:include filename="package://comau_racer5_080_description/urdf/materials.xacro"/> -->
+    <xacro:macro name="inertial_box" params="mass x y z *origin">
+        <inertial>
+            <xacro:insert_block name="origin"/>
+            <mass value="${mass}" />
+            <inertia ixx="${(1/12) * mass * (y*y+z*z)}" ixy="0.0" ixz="0.0" iyy="${(1/12) * mass * (x*x+z*z)}" iyz="0.0" izz="${(1/12) * mass * (x*x+y*y)}" />
+        </inertial>
+    </xacro:macro>
+    <link name="world"></link>
     <xacro:property name="r2d" value="${pi/180}"/>
     <xacro:property name="meshes_path" value="package://comau_racer5_080_description/meshes"/>
@@ -12,5 +21,19 @@
             <material name="grey"/>
         </visual>
-    </link>
+        <collision>
+            <origin xyz="0.0 0.0 0.0" rpy="0.0 0.0 0.0"/>
+            <geometry>
+                <box size="0.2 0.2 0.2"/>
+            </geometry>
+        </collision>
+        <xacro:inertial_box mass="0.1" x="0.12" y="0.15" z="0.15">
+            <origin xyz="0.0 0 0" rpy="0 0 0"/>
+        </xacro:inertial_box>
+    </link>
+    <joint name="base_joint" type="fixed">
+        <origin xyz="1.5 1.0 0" rpy="0 0 0"/>
+        <parent link="world"/>
+        <child link="base_link"/>
+    </joint>
     <link name="q1_link">
         <visual>
@@ -21,10 +44,27 @@
             <material name="grey"/>
         </visual>
+        <collision>
+            <origin xyz="0.0 0 0" rpy="0 0 0"/>
+            <geometry>
+                <box size="0.12 0.15 0.15" />
+            </geometry>
+        </collision>
+        <!-- <xacro:inertial_box mass="0.1" x="0.12" y="0.15" z="0.15">
+            <origin xyz="0.0 0 0" rpy="0 0 0"/>
+        </xacro:inertial_box> -->
+        <inertial>
+            <mass value="1"/>
+            <inertia
+              ixx="1.0" ixy="0.0" ixz="0.0"
+              iyy="1.0" iyz="0.0"
+              izz="1.0"/>
+      </inertial>
     </link>
     <joint name="q1_joint" type="revolute">
+        <origin xyz="0 0 0" rpy="0 0 0"/>
+        <parent link="base_link"/>
+        <child link="q1_link"/>
         <axis xyz="0 0 1"/>
-       <parent link="base_link"/>
-       <child link="q1_link"/>
-       <limit lower="-${r2d*170}" upper="${r2d*170}" effort="0.0" velocity="${r2d*400}"/>
+        <limit lower="-${r2d*170}" upper="${r2d*170}" effort="0.0" velocity="${r2d*400}"/>
     </joint>
     <link name="q2_link">
@@ -36,11 +76,24 @@
             <material name="grey"/>
         </visual>
+        <collision>
+            <origin xyz="0.0 0 0" rpy="0 0 0"/>
+            <geometry>
+                <box size="0.12 0.15 0.15" />
+            </geometry>
+        </collision>
+        <inertial>
+            <mass value="1"/>
+            <inertia
+              ixx="1.0" ixy="0.0" ixz="0.0"
+              iyy="1.0" iyz="0.0"
+              izz="1.0"/>
+      </inertial>
     </link>
     <joint name="q2_joint" type="revolute">
-       <axis xyz="0 1 0"/>
-       <origin xyz="0.050 0.0 0.365"/>
-       <parent link="q1_link"/>
-       <child link="q2_link"/>
-       <limit lower="-${r2d*85}" upper="${r2d*135}" effort="0.0" velocity="${r2d*360}"/>
+        <axis xyz="0 1 0"/>
+        <origin xyz="0.050 0.0 0.365"/>
+        <parent link="q1_link"/>
+        <child link="q2_link"/>
+        <limit lower="-${r2d*85}" upper="${r2d*135}" effort="0.0" velocity="${r2d*360}"/>
     </joint>
     <link name="q3_link">
@@ -52,4 +105,17 @@
             <material name="grey"/>
         </visual>
+        <collision>
+            <origin xyz="0.0 0 0" rpy="0 0 0"/>
+            <geometry>
+                <box size="0.12 0.15 0.15" />
+            </geometry>
+        </collision>
+        <inertial>
+            <mass value="1"/>
+            <inertia
+              ixx="1.0" ixy="0.0" ixz="0.0"
+              iyy="1.0" iyz="0.0"
+              izz="1.0"/>
+      </inertial>
     </link>
     <joint name="q3_joint" type="revolute">
@@ -68,4 +134,17 @@
             <material name="grey"/>
         </visual>
+        <collision>
+            <origin xyz="0.0 0 0" rpy="0 0 0"/>
+            <geometry>
+                <box size="0.12 0.15 0.15" />
+            </geometry>
+        </collision>
+        <inertial>
+            <mass value="1"/>
+            <inertia
+              ixx="1.0" ixy="0.0" ixz="0.0"
+              iyy="1.0" iyz="0.0"
+              izz="1.0"/>
+      </inertial>
     </link>
     <joint name="q4_joint" type="revolute">
@@ -84,4 +163,17 @@
             <material name="grey"/>
         </visual>
+        <collision>
+            <origin xyz="0.0 0 0" rpy="0 0 0"/>
+            <geometry>
+                <box size="0.12 0.15 0.15" />
+            </geometry>
+        </collision>
+        <inertial>
+            <mass value="1"/>
+            <inertia
+              ixx="1.0" ixy="0.0" ixz="0.0"
+              iyy="1.0" iyz="0.0"
+              izz="1.0"/>
+      </inertial>
     </link>
     <joint name="q5_joint" type="revolute">
@@ -100,4 +192,17 @@
             <material name="grey"/>
         </visual>
+        <collision>
+            <origin xyz="0.0 0 0" rpy="0 0 0"/>
+            <geometry>
+                <box size="0.12 0.15 0.15" />
+            </geometry>
+        </collision>
+        <inertial>
+            <mass value="1"/>
+            <inertia
+              ixx="1.0" ixy="0.0" ixz="0.0"
+              iyy="1.0" iyz="0.0"
+              izz="1.0"/>
+      </inertial>
     </link>
     <joint name="q6_joint" type="revolute">
@@ -108,3 +213,30 @@
        <limit lower="-${r2d*2700}" upper="${r2d*2700}" effort="0.0" velocity="${r2d*800}"/>
     </joint>
+    <!-- Gazebo requires the use of plugins to interact with other systems such as ROS. -->
+    <!-- This plugin will publish the joint_states for the selected joints
+            (which robot_state_publisher can then use to broadcast the approprate tf). -->
+    <gazebo>
+        <plugin name="gazebo_ros_joint_state_publisher" filename="libgazebo_ros_joint_state_publisher.so">
+            <update_rate>20</update_rate>
+            <joint_name>q1_joint</joint_name>
+            <joint_name>q2_joint</joint_name>
+            <joint_name>q3_joint</joint_name>
+            <joint_name>q4_joint</joint_name>
+            <joint_name>q5_joint</joint_name>
+            <joint_name>q6_joint</joint_name>
+        </plugin>
+    </gazebo>
+    <gazebo>
+    </gazebo>
+    <!-- This plugin will read a JointTrajectory message from the /set_joint_trajectory topic
+            and move the machine accordingly. It's a bit clunky but it works. -->
+    <!-- You'll probably want to add damping to the joints to stop them it flopping around.
+            e.g. <dynamics damping="10.0" friction="10.0"/> -->
+    <!-- Here's an example message to publish to test it:
+            ros2 topic pub -1 /set_joint_trajectory trajectory_msgs/msg/JointTrajectory  '{header: {frame_id: world}, joint_names: [slider_joint, arm_joint], points: [  {positions: {0.8,0.6}} ]}' -->
+    <gazebo>
+        <plugin name="gazebo_ros_joint_pose_trajectory" filename="libgazebo_ros_joint_pose_trajectory.so">
+            <update_rate>2</update_rate>
+        </plugin>
+    </gazebo>
 </robot>

File: urdf/materials.xacro (robot description, xacro)
@@ -1,27 +1,27 @@
 <?xml version="1.0"?>
 <robot xmlns:xacro="http://www.ros.org/wiki/xacro">
-    <material name="black">
-        <color rgba="0.0 0.0 0.0 1.0"/>
-      </material>
-      <material name="blue">
-        <color rgba="0.0 0.0 0.8 1.0"/>
-      </material>
-      <material name="green">
-        <color rgba="0.0 1.0 0.0 1.0"/>
-      </material>
-      <material name="grey">
-        <color rgba="0.2 0.2 0.2 1.0"/>
-      </material>
-      <material name="orange">
-        <color rgba="${255/255} ${108/255} ${10/255} 1.0"/>
-      </material>
-      <material name="brown">
-        <color rgba="${222/255} ${207/255} ${195/255} 1.0"/>
-      </material>
-      <material name="red">
-        <color rgba="0.8 0.0 0.0 1.0"/>
-      </material>
-      <material name="white">
-        <color rgba="1.0 1.0 1.0 1.0"/>
-      </material>
+  <material name="black">
+    <color rgba="0.0 0.0 0.0 1.0"/>
+  </material>
+  <material name="blue">
+    <color rgba="0.0 0.0 0.8 1.0"/>
+  </material>
+  <material name="green">
+    <color rgba="0.0 1.0 0.0 1.0"/>
+  </material>
+  <material name="grey">
+    <color rgba="0.2 0.2 0.2 1.0"/>
+  </material>
+  <material name="orange">
+    <color rgba="${255/255} ${108/255} ${10/255} 1.0"/>
+  </material>
+  <material name="brown">
+    <color rgba="${222/255} ${207/255} ${195/255} 1.0"/>
+  </material>
+  <material name="red">
+    <color rgba="0.8 0.0 0.0 1.0"/>
+  </material>
+  <material name="white">
+    <color rgba="1.0 1.0 1.0 1.0"/>
+  </material>
 </robot>
